Commit message: 説明を追加

File: whill_vehicle_description/urdf/vehicle.xacro (robot description, xacro)
@@ -4,11 +4,12 @@
   <xacro:property name="vehicle_info" value="${xacro.load_yaml('$(find whill_vehicle_description)/config/vehicle_info.param.yaml')}"/>
   <!-- vehicle body -->
+  <!-- TODO: 時間に余裕があればwhillのdaeを作成する -->
   <link name="base_link">
-    <visual>
+    <!-- <visual>
       <origin xyz="${vehicle_info['/**']['ros__parameters']['wheel_base']/2.0} 0 0" rpy="${pi/2.0} 0 ${pi}"/>
       <geometry>
         <mesh filename="package://whill_vehicle_description/mesh/lexus.dae" scale="1 1 1"/>
       </geometry>
-    </visual>
+    </visual> -->
   </link>
 </robot>
