Commit message: refactor: rename whill to canedudev_rover

File: canedudev_rover_vehicle_description/urdf/vehicle.xacro (robot description, xacro)
@@ -2,12 +2,12 @@
 <robot xmlns:xacro="http://ros.org/wiki/xacro">
   <!-- load parameter -->
-  <xacro:property name="vehicle_info" value="${xacro.load_yaml('$(find whill_vehicle_description)/config/vehicle_info.param.yaml')}"/>
+  <xacro:property name="vehicle_info" value="${xacro.load_yaml('$(find canedudev_rover_vehicle_description)/config/vehicle_info.param.yaml')}"/>
   <!-- vehicle body -->
-  <!-- TODO: 時間に余裕があればwhillのdaeを作成する -->
+  <!-- TODO: 時間に余裕があればcanedudev_roverのdaeを作成する -->
   <link name="base_link">
     <!-- <visual>
       <origin xyz="${vehicle_info['/**']['ros__parameters']['wheel_base']/2.0} 0 0" rpy="${pi/2.0} 0 ${pi}"/>
       <geometry>
-        <mesh filename="package://whill_vehicle_description/mesh/lexus.dae" scale="1 1 1"/>
+        <mesh filename="package://canedudev_rover_vehicle_description/mesh/lexus.dae" scale="1 1 1"/>
       </geometry>
     </visual> -->
